File: yagi.sch (KiCad schematic (older format))
At the start: 22 parts, among them P1 CONN_01X01, P2 CONN_01X01, P3 CONN_01X01, P4 CONN_01X01, Q1 Q_NPN_BCE, Q2 Q_NPN_BCE, Q3 Q_NPN_BCE

Commit message: Layouting
Parts:
- removed 15uH1: IND, symbol IND
- removed P2: CONN_01X01, symbol CONN_01X01
- removed Q1, Q2, Q3: Q_NPN_BCE, symbol Q_NPN_BCE
- removed R7: 5.1M, symbol R
- added C1: 220uF, Capacitors_SMD:c_elec_6.3x7.7, symbol CP
- added C3: 1uF, Capacitors_SMD:C_0603, symbol C
- added C6, C9: 0.1uF, Capacitors_SMD:C_0805, symbol C
- added C7: 22uF, Capacitors_SMD:c_elec_5x4.5, symbol CP
- added C8: 1uF, Capacitors_SMD:C_0805, symbol C
- added D1, D2, D4, D5, D6, D7: Led_Small, LEDs:LED-0603, symbol Led_Small
- added IC1: AT24CS32-SSHM, Housings_SOIC:SOIC-8_3.9x4.9mm_Pitch1.27mm, symbol AT24CS32-SSHM
- added J1: RPi_GPIO, RPi_Hat:Pin_Header_Straight_2x20, symbol RPi_GPIO
- added L1: 15mH, chenit:SRR0908-Y, symbol SRR0908-Y
- added P3: CONN_01X01, Wire_Pads:SolderWirePad_single_0-8mmDrill, symbol CONN_01X01
- added P5, P7: CONN_01X02, Pin_Headers:Pin_Header_Straight_1x02, symbol CONN_01X02
- added P6: CONN_01X03, Pin_Headers:Pin_Header_Straight_1x03, symbol CONN_01X03
- added Q1, Q2: STN0214, chenit:SOT223, symbol Q_NPN_BCEC
- added Q3: MMBT4401, TO_SOT_Packages_SMD:SOT-23, symbol Q_NPN_BEC
- added R1, R15, R16, R17, R18, R2: R, Resistors_SMD:R_0805_HandSoldering, symbol R
- added R12: 1k, Resistors_SMD:R_0805_HandSoldering, symbol R
- added R13, R14: 3.9k, Resistors_SMD:R_0805_HandSoldering, symbol R
- added R19, R20, R21, R22: 10k, Resistors_SMD:R_0805_HandSoldering, symbol R
- added U1: 74LS244, Housings_SOIC:SOIC-20_7.5x12.8mm_Pitch1.27mm, symbol 74LS244
- C2: renamed from C1; value C -> 47nF; footprint (none) -> Capacitors_SMD:C_0805
- C4: renamed from C2; value C -> 47nF; footprint (none) -> Capacitors_SMD:C_0805
- C5: renamed from C3; value C -> 330pF; footprint (none) -> Capacitors_SMD:C_0603
- D3: renamed from D1; value D -> RFU02VSM8STR; footprint (none) -> chenit:TUMD2SM
- P1: value CONN_01X01 -> HV+; footprint (none) -> Wire_Pads:SolderWirePad_single_1-2mmDrill
- P2: renamed from P3; value CONN_01X01 -> HV-; footprint (none) -> Wire_Pads:SolderWirePad_single_1-2mmDrill
- P4: footprint (none) -> Wire_Pads:SolderWirePad_single_0-8mmDrill
- R10: renamed from R9; footprint (none) -> Resistors_SMD:R_0805_HandSoldering
- R11: renamed from R10; footprint (none) -> Resistors_SMD:R_0805_HandSoldering
- R3: renamed from R1; footprint (none) -> Resistors_SMD:R_0805_HandSoldering
- R4: renamed from R2; footprint (none) -> Resistors_SMD:R_0805_HandSoldering
- R5: renamed from R3; footprint (none) -> Resistors_SMD:R_0805_HandSoldering
- R6: renamed from R4; footprint (none) -> Resistors_SMD:R_0805_HandSoldering
- R7: renamed from R5; footprint (none) -> Resistors_SMD:R_0805_HandSoldering
- R8: renamed from R6; footprint (none) -> Resistors_SMD:R_0805_HandSoldering
- R9: renamed from R8; footprint (none) -> Resistors_SMD:R_0805_HandSoldering
Connections:
- net +3V3: now also C6.1, C7.1, C8.1, C9.1, IC1.8 (VCC), J1.1 (3.3V), R12.1, R13.1, R14.1, U1.20 (VCC)
- net +5V: now also C1.1, C3.1, J1.2 (5V), J1.4 (5V)
- net GND: now also C1.2, C3.2, C6.2, C7.2, C8.2, C9.2, D1.1 (K), D2.1 (K), D4.1 (K), D5.1 (K), D6.1 (K), D7.1 (K), IC1.1 (A0), IC1.2 (A1), IC1.3 (A2), IC1.4 (GND), J1.6 (GND), J1.9 (GND), P5.1 (P1), Q1.3 (E), Q2.3 (E), Q3.2 (E), U1.1 (OEa), U1.10 (GND), U1.19 (OEb)
- net discharge: now also R2.2, U1.7 (O1b)
- net pulse: now also R1.2, U1.9 (O0b)
- net at D3.2 (A): now also L1.5, L1.6, L1.7, L1.8, Q1.2 (C), Q1.4 (C)
- net at R6.1, R7.2: now also Q2.2 (C), Q2.4 (C)
- net at C4.1, R7.1: now also R8.1; no longer R8.2
- net at R5.1: now also L1.1, L1.2, L1.3, L1.4
- net at R3.1: now also Q1.1 (B)
- net at P1.1 (P1): now also R8.2; no longer R8.1
- net at R4.1: now also Q2.1 (B)
- net at R10.2, R9.1: now also P3.1 (P1), Q3.1 (B)
- net detect: now reaches P4.1 (P1), R11.1
- net detect: now also Q3.3 (C), U1.2 (I0a)
- new net: R18.1, R22.2, U1.12 (O3a)
- new net: R17.1, R21.2, U1.14 (O2a)
- new net: R16.1, R20.2, U1.16 (O1a)
- new net: R15.1, R19.2, U1.18 (O0a)
- new net: P7.2 (P2), U1.3 (O3b)
- new net: P6.3 (P3), U1.4 (I1a)
- new net: P7.1 (P1), U1.5 (O2b)
- new net: P6.2 (P2), U1.6 (I2a)
- new net: P6.1 (P1), U1.8 (I3a)
- new net: IC1.7 (WP), P5.2 (P2), R12.2
- new net: D1.2 (A), R1.1
- new net: D2.2 (A), R2.1
- new net: D7.2 (A), R18.2
- new net: D6.2 (A), R17.2
- new net: D4.2 (A), R15.2
- new net: D5.2 (A), R16.2
- new net AUX_IN1: J1.36 (GPIO16), R20.1
- new net AUX_IN2: J1.38 (GPIO20), R21.1
- new net AUX_IN3: J1.40 (GPIO21), R22.1
- new net AUX_OUT1: J1.16 (GPIO23), U1.15 (I2b)
- new net AUX_OUT2: J1.18 (GPIO24), U1.17 (I3b)
- new net DET: J1.32 (GPIO12), R19.1
- new net DISC: J1.14 (GND), U1.13 (I1b)
- new net ID_SC: IC1.6 (SCL), J1.28 (ID_SC), R14.2
- new net ID_SD: IC1.5 (SDA), J1.27 (ID_SD), R13.2
- new net PWM: J1.12 (GPIO18), U1.11 (I0b)
Other:
- moved on the sheet: C2, C4, C5, D3, P1, P2, P4, R10, R11, R3, R4, R5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
