File: yagi.kicad_pcb (KiCad board)
At the start: 2 copper layers, 65 x 56 mm, 76 parts, among them IC1 AT24CS32-SSHM, J1 RPi_GPIO, P1 CONN_01X03, P10 CONN_01X02, P11 CONN_01X03, P12 CONN_01X03, P13 CONN_01X03, P14 CONN_01X03, P15 CONN_01X02, P16 CONN_01X02, P17 CONN_01X02, P2 CONN_01X01, P3 CONN_01X01, P4 CONN_01X02, P5 HV+, P6 CONN_01X02, P7 HV-, P8 CONN_01X01, P9 CONN_01X01, Q1 MMBT4401, Q2 STN0214, Q3 STN0214, Q4 MMBT4401, U1 TLC555, U2 74LS244

Commit message: Renamed files according to seeed guidelines.
Routing:
- net GND: vias 16 -> 6
- net (no net): vias 0 -> 10
Changed lines of the file:
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@@
   (gr_line (start 41.5 91) (end 100.5 91) (angle 90) (layer Edge.Cuts) (width 0.1))
   (gr_line (start 103.5 37.5) (end 103.5 88) (angle 90) (layer Edge.Cuts) (width 0.1))
-  (via (at 72.39 46.99) (size 0.6) (drill 0.4) (layers F.Cu B.Cu) (net 1))
-  (via (at 71.12 46.99) (size 0.6) (drill 0.4) (layers F.Cu B.Cu) (net 1))
-  (via (at 73.025 46.355) (size 0.6) (drill 0.4) (layers F.Cu B.Cu) (net 1))
-  (via (at 71.755 46.355) (size 0.6) (drill 0.4) (layers F.Cu B.Cu) (net 1))
-  (via (at 70.485 46.355) (size 0.6) (drill 0.4) (layers F.Cu B.Cu) (net 1))
-  (via (at 86.995 45.72) (size 0.6) (drill 0.4) (layers F.Cu B.Cu) (net 1))
-  (via (at 86.995 44.45) (size 0.6) (drill 0.4) (layers F.Cu B.Cu) (net 1))
-  (via (at 86.995 51.435) (size 0.6) (drill 0.4) (layers F.Cu B.Cu) (net 1))
-  (via (at 85.09 51.435) (size 0.6) (drill 0.4) (layers F.Cu B.Cu) (net 1))
-  (via (at 83.185 51.435) (size 0.6) (drill 0.4) (layers F.Cu B.Cu) (net 1))
+  (via (at 72.39 46.99) (size 0.6) (drill 0.4) (layers F.Cu B.Cu) (net 0))
+  (via (at 71.12 46.99) (size 0.6) (drill 0.4) (layers F.Cu B.Cu) (net 0))
+  (via (at 73.025 46.355) (size 0.6) (drill 0.4) (layers F.Cu B.Cu) (net 0))
+  (via (at 71.755 46.355) (size 0.6) (drill 0.4) (layers F.Cu B.Cu) (net 0))
+  (via (at 70.485 46.355) (size 0.6) (drill 0.4) (layers F.Cu B.Cu) (net 0))
+  (via (at 86.995 45.72) (size 0.6) (drill 0.4) (layers F.Cu B.Cu) (net 0))
+  (via (at 86.995 44.45) (size 0.6) (drill 0.4) (layers F.Cu B.Cu) (net 0))
+  (via (at 86.995 51.435) (size 0.6) (drill 0.4) (layers F.Cu B.Cu) (net 0))
+  (via (at 85.09 51.435) (size 0.6) (drill 0.4) (layers F.Cu B.Cu) (net 0))
+  (via (at 83.185 51.435) (size 0.6) (drill 0.4) (layers F.Cu B.Cu) (net 0))
   (segment (start 70.485 58.42) (end 69.85 59.055) (width 1) (layer B.Cu) (net 1))
   (segment (start 69.85 59.055) (end 62.865 59.055) (width 1) (layer B.Cu) (net 1))
@@
   (segment (start 61.849 58.039) (end 60.706 58.039) (width 1) (layer B.Cu) (net 1))
   (segment (start 62.865 59.055) (end 61.849 58.039) (width 1) (layer B.Cu) (net 1))
-  (segment (start 71.435 77.73924) (end 72.62876 77.73924) (width 1) (layer B.Cu) (net 1) (status 400000))
-  (segment (start 73.025 77.343) (end 73.025 79.375) (width 1) (layer F.Cu) (net 1) (status 800000))
+  (segment (start 71.435 77.73924) (end 72.62876 77.73924) (width 1) (layer B.Cu) (net 1))
+  (segment (start 73.025 77.343) (end 73.025 79.375) (width 1) (layer F.Cu) (net 1))
   (via (at 73.025 77.343) (size 0.6) (drill 0.4) (layers F.Cu B.Cu) (net 1))
   (segment (start 72.62876 77.73924) (end 73.025 77.343) (width 1) (layer B.Cu) (net 1))
-  (segment (start 98.11 73.66) (end 93.345 73.66) (width 0.5) (layer F.Cu) (net 1) (status 400000))
-  (segment (start 92.075 72.39) (end 92.075 63.58) (width 0.5) (layer F.Cu) (net 1) (status 800000))
+  (segment (start 98.11 73.66) (end 93.345 73.66) (width 0.5) (layer F.Cu) (net 1))
+  (segment (start 92.075 72.39) (end 92.075 63.58) (width 0.5) (layer F.Cu) (net 1))
   (segment (start 93.345 73.66) (end 92.075 72.39) (width 0.5) (layer F.Cu) (net 1))
   (segment (start 97.47 56.14924) (end 97.47 55.56) (width 0.5) (layer B.Cu) (net 1))
@@
   (segment (start 56.515 73.025) (end 58.54 73.025) (width 0.5) (layer F.Cu) (net 2))
   (segment (start 55.88 73.66) (end 56.515 73.025) (width 0.5) (layer F.Cu) (net 2))
-  (segment (start 47.09 62.29) (end 45.593 60.793) (width 1) (layer F.Cu) (net 3) (status 400000))
+  (segment (start 47.09 62.29) (end 45.593 60.793) (width 1) (layer F.Cu) (net 3))
   (segment (start 45.593 60.793) (end 45.593 57.658) (width 1) (layer F.Cu) (net 3))
   (via (at 45.72 69.85) (size 0.6) (drill 0.4) (layers F.Cu B.Cu) (net 3))
@@
   (segment (start 57.15 81.915) (end 57.15 84.455) (width 0.5) (layer B.Cu) (net 3))
   (segment (start 57.785 80.645) (end 57.15 81.28) (width 0.5) (layer B.Cu) (net 3))
-  (segment (start 100.01 73.66) (end 100.01 65.085) (width 0.5) (layer F.Cu) (net 4) (status 400000))
-  (segment (start 98.505 63.58) (end 94.615 63.58) (width 0.5) (layer F.Cu) (net 4) (status 800000))
+  (segment (start 100.01 73.66) (end 100.01 65.085) (width 0.5) (layer F.Cu) (net 4))
+  (segment (start 98.505 63.58) (end 94.615 63.58) (width 0.5) (layer F.Cu) (net 4))
   (segment (start 100.01 65.085) (end 98.505 63.58) (width 0.5) (layer F.Cu) (net 4))
-  (segment (start 100.01 73.66) (end 100.01 74.61) (width 0.5) (layer F.Cu) (net 4) (status 400000))
-  (segment (start 100.33 74.93) (end 100.33 77.47) (width 0.5) (layer F.Cu) (net 4) (status 800000))
+  (segment (start 100.01 73.66) (end 100.01 74.61) (width 0.5) (layer F.Cu) (net 4))
+  (segment (start 100.33 74.93) (end 100.33 77.47) (width 0.5) (layer F.Cu) (net 4))
   (segment (start 100.01 74.61) (end 100.33 74.93) (width 0.5) (layer F.Cu) (net 4))
-  (segment (start 100.33 73.98) (end 100.01 73.66) (width 0.5) (layer F.Cu) (net 4) (status C00000))
+  (segment (start 100.33 73.98) (end 100.01 73.66) (width 0.5) (layer F.Cu) (net 4))
   (segment (start 56.515 58.07964) (end 61.88964 58.07964) (width 1) (layer F.Cu) (net 5))
   (segment (start 61.88964 58.07964) (end 62.865 59.055) (width 1) (layer F.Cu) (net 5))
